File: CompactMotor.kicad_pcb (KiCad board)
At the start: 4 copper layers, 39.4 x 41.3 mm, 44 parts, among them J1 Conn_01x04_Male, J3 Conn_01x02_Female, J5 Conn_01x01_Male, J6 Conn_01x01_Male, J7 Conn_01x01_Male, J8 Conn_01x01_Male, U1 ESP32-WROOM-32D, U2 AMS1117-3.3, U3 TMC2130-TA

Commit message: CLP BOM
Parts:
- removed the J3 at (14.7, 15.1)
- removed JP3: SolderJumper_2_Open, Jumper:SolderJumper-2_P1.3mm_Open_TrianglePad1.0x1.5mm
- added ?: , , F.Cu at (34.8, 44.8)
- added ?: , , F.Cu at (21.3, 45.0)
- added ?: , , F.Cu at (1.02, 40.1)
- added ?: , , F.Cu at (34.7, -3.81)
- added ?: , , F.Cu at (21.6, -3.94)
- added ?: , , F.Cu at (30.9, 40.0)
- added J2: Conn_01x02_Male, Connector_PinHeader_2.54mm:PinHeader_1x02_P2.54mm_Horizontal, B.Cu at (4.45, 4.57)
- added REF**: MountingHole_2.5mm_Pad, MountingHole:MountingHole_2.5mm_Pad, F.Cu at (30.5, 1.52)
- added SW1: SW_Push, CompactMotor:SW1AB-260-10T28, B.Cu at (15.2, 14.6)
- added TP1: TestPoint, TestPoint:TestPoint_Pad_4.0x4.0mm, F.Cu at (22.9, 20.6)
- D1: footprint LED_SMD:LED_0201_0603Metric -> LED_SMD:LED_0402_1005Metric
- D2: value LED -> LED Red; footprint LED_SMD:LED_0201_0603Metric -> LED_SMD:LED_0402_1005Metric
- D3: value LED -> LED Blue; footprint LED_SMD:LED_0201_0603Metric -> LED_SMD:LED_0402_1005Metric
- J1, J5, J6, J7, J8: moved to B.Cu
- J3: footprint Connector_PinHeader_2.54mm:PinHeader_1x02_P2.54mm_Vertical -> Connector_PinHeader_2.54mm:PinHeader_1x02_P2.54mm_Horizontal; moved to B.Cu
- R7: value R2k -> R150
- R8: value R2k -> R100
- moved J3 27.0 mm to (4.45, 34.2), turned to 180 degrees
- moved C11 10.1 mm to (12.6, 33.3)
- moved C10 9.79 mm to (13.1, 36.1), turned to -90 degrees
- moved J1 7.75 mm to (22.9, 2.79)
- moved D3 5.21 mm to (3.43, 9.78)
- moved R8 5.21 mm to (1.65, 9.78)
- moved C9 4.82 mm to (7.87, 32.4)
- moved J5 4.20 mm to (29.2, -2.41)
- moved J6 4.15 mm to (30.2, 43.4)
- moved D2 3.81 mm to (7.11, 9.78)
- moved R7 3.81 mm to (5.33, 9.78)
- moved R6 1.90 mm to (5.21, 32.4)
- moved U2 0.51 mm to (18.5, 35.6)
Connections:
- U3 pad 13: Net-(J1-Pad1) -> Net-(J1-Pad4)
- U3 pad 15: Net-(J1-Pad2) -> Net-(J1-Pad3)
- U3 pad 32: Net-(J1-Pad3) -> Net-(J1-Pad2)
- U3 pad 34: Net-(J1-Pad4) -> Net-(J1-Pad1)
Routing:
- net Net-(J1-Pad2): track 17.3 -> 50.0 mm
- net Net-(J1-Pad3): track 50.0 -> 18.1 mm
- net Net-(J1-Pad1): track 17.9 -> 49.4 mm, vias 0 -> 1
- net Net-(J1-Pad4): track 49.4 -> 18.5 mm, vias 1 -> 0
- net IO0: track 8.47 -> 39.1 mm, vias 1 -> 2
- net RXD0: track 0.00 -> 26.1 mm
- net TXD0: track 0.00 -> 21.0 mm
- net GNDREF: track 44.3 -> 61.1 mm, vias 97 -> 95
- net 3V3: track 41.9 -> 47.6 mm
- net EN: track 34.8 -> 40.0 mm
- net Net-(R8-Pad1): track 10.9 -> 5.78 mm
- net STALLMINUS: track 26.7 -> 30.7 mm
- net 5V0: track 19.7 -> 23.4 mm, vias 6 -> 7
- net Net-(R7-Pad1): track 2.64 -> 5.50 mm
- net VM: track 73.1 -> 74.4 mm
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- added copper zone on F.Cu, net GNDREF
- added copper zone on In2.Cu, net GNDREF
Other:
- board size 39.4 x 41.3 mm -> 43.4 x 51.2 mm
- board text added: "5V0"
- board text added: "GND"
- board text added: "IO0"
- board text added: "OA1"
- board text added: "OA2"
- board text added: "OB1"
- board text added: "OB2"
- board text added: "RXD0"
- board text added: "STALL+"
- board text added: "STALL-"
- board text added: "TXD0"
