File: CompactMotor.kicad_sch (KiCad schematic)
At the start: 25 parts, among them J1 Conn_01x04_Male, J2 Conn_01x01_Female, U1 ESP32-WROOM-32D, U2 AMS1117-3.3, U3 TMC2130-TA

Commit message: Only trx-rx
Parts:
- removed J2: Conn_01x01_Female, Connector_PinHeader_2.54mm:PinHeader_1x01_P2.54mm_Vertical, symbol Connector:Conn_01x01_Female
- added C14: C100nF, Capacitor_SMD:C_0603_1608Metric, symbol Device:C
- added C15: C1uF, Capacitor_SMD:C_0603_1608Metric, symbol Device:C
- added D2, D3: LED, LED_SMD:LED_0201_0603Metric, symbol Device:LED
- added J3: Conn_01x02_Female, Connector_PinHeader_2.54mm:PinHeader_1x02_P2.54mm_Vertical, symbol Connector:Conn_01x02_Female
- added J5, J6, J7, J8: Conn_01x01_Male, Connector_PinHeader_2.54mm:PinHeader_1x01_P2.54mm_Horizontal, symbol Connector:Conn_01x01_Male
- added JP1, JP2: SolderJumper_3_Open, Jumper:SolderJumper-3_P1.3mm_Open_RoundedPad1.0x1.5mm, symbol Jumper:SolderJumper_3_Open
- added JP3: SolderJumper_2_Open, Jumper:SolderJumper-2_P1.3mm_Open_TrianglePad1.0x1.5mm, symbol Jumper:SolderJumper_2_Open
- added R7, R8: R2k, Resistor_SMD:R_0402_1005Metric, symbol Device:R
Connections:
- net IO27 is gone; now on net DC0: U1.12 (IO27)
- net IO34 is gone; now on net DIAG0: U1.6 (IO34)
- net IO35 is gone; now on net DIAG1: U1.7 (IO35)
- net 5V0: now also C4.2, U3.8 (VCC_IO), J5.1 (Pin_1), J7.1 (Pin_1)
- net DCEN_CFG4: now also JP1.1 (A)
- net DCIN_CFG5: now also JP2.1 (A)
- net EN: now also JP3.1 (A)
- net GNDREF: now also C14.2, C15.1, D2.1 (K), D3.1 (K), J3.1 (Pin_1), JP1.3 (B), JP2.3 (B), JP3.2 (B)
- net VM: now also C8.2, U3.30 (VSA), U3.31 (VS), C14.1, C15.2
- net at J1.1 (Pin_1): now also U3.13 (OB1); no longer U3.15 (OB2)
- net at J1.2 (Pin_2): now also U3.15 (OB2); no longer U3.13 (OB1)
- net at C5.2, R3.1, U3.26 (VCC): no longer C4.2, U3.8 (VCC_IO)
- net IO21: no longer names the net of U1.33 (IO21)
- net IO21: now also R7.1
- net IO22: no longer names the net of U1.36 (IO22)
- net IO22: now also R8.1
- net IO25 renamed STALLPLUS
- net STALLPLUS: now also J8.1 (Pin_1)
- net IO26 renamed STALLMINUS
- net STALLMINUS: now also J6.1 (Pin_1)
- net IO32: no longer names the net of U1.8 (IO32)
- net IO32: now also JP1.2 (C)
- net IO33: no longer names the net of U1.9 (IO33)
- net IO33: now also JP2.2 (C)
- net SD0 renamed IO0
- net IO0: now also J3.2 (Pin_2)
- new net: D2.2 (A), R7.2
- new net: D3.2 (A), R8.2

Commit message: CLP BOM
Parts:
- removed JP3: SolderJumper_2_Open, Jumper:SolderJumper-2_P1.3mm_Open_TrianglePad1.0x1.5mm, symbol Jumper:SolderJumper_2_Open
- added J2: Conn_01x02_Male, Connector_PinHeader_2.54mm:PinHeader_1x02_P2.54mm_Horizontal, symbol Connector:Conn_01x02_Male
- added SW1: SW_Push, CompactMotor:SW1AB-260-10T28, symbol Switch:SW_Push
- added TP1: TestPoint, TestPoint:TestPoint_Pad_4.0x4.0mm, symbol Connector:TestPoint
- D1: footprint LED_SMD:LED_0201_0603Metric -> LED_SMD:LED_0402_1005Metric
- D2: value LED -> LED Red; footprint LED_SMD:LED_0201_0603Metric -> LED_SMD:LED_0402_1005Metric
- D3: value LED -> LED Blue; footprint LED_SMD:LED_0201_0603Metric -> LED_SMD:LED_0402_1005Metric
- J3: footprint Connector_PinHeader_2.54mm:PinHeader_1x02_P2.54mm_Vertical -> Connector_PinHeader_2.54mm:PinHeader_1x02_P2.54mm_Horizontal
- R7: value R2k -> R150
- R8: value R2k -> R100
Connections:
- net EN: now also SW1.1
- net GNDREF: now also SW1.2, TP1.1
- net RXD0: now also J2.1 (Pin_1)
- net TXD0: now also J2.2 (Pin_2)
- net at J1.1 (Pin_1): now also U3.34 (OA1); no longer U3.13 (OB1)
- net at J1.2 (Pin_2): now also U3.32 (OA2); no longer U3.15 (OB2)
- net at J1.3 (Pin_3): now also U3.15 (OB2); no longer U3.32 (OA2)
- net at J1.4 (Pin_4): now also U3.13 (OB1); no longer U3.34 (OA1)
Other:
- moved on the sheet: J1
